File: speedometer.kicad_pcb (KiCad board)
At the start: 2 copper layers, 100 x 100 mm, 40 parts, among them J1 Conn_01x03, J2 Conn_01x03, J3 Conn_01x03, J4 Conn_01x03, Q1 SSM3J332R, Q2 MMBT3904, Q3 MMBT3904, Q4 MMBT3904, Q5 L-51ROPT1D1, Q6 TMBT3906, Q7 TMBT3906, Q8 L-51ROPT1D1, Q9 TMBT3906, SW1 SW_Push, SW2 RESET_SW, U1 RaspberryPi-Pico, U2 OSL30561-IRA

Commit message: アートワーク完成
Parts:
- added H5: MountingHole, myLib:MountingHole_3.2mm_M3_noResist, F.Cu at (7.50, 15.0)
- added H6: MountingHole, myLib:MountingHole_3.2mm_M3_noResist, F.Cu at (7.50, 85.0)
- added H7: MountingHole, myLib:MountingHole_3.2mm_M3_noResist, F.Cu at (92.5, 15.0)
- added H8: MountingHole, myLib:MountingHole_3.2mm_M3_noResist, F.Cu at (92.5, 85.0)
- added R14: 470R, Resistor_SMD:R_0603_1608Metric, B.Cu at (43.0, 6.00)
- added R15: 470R, Resistor_SMD:R_0603_1608Metric, B.Cu at (50.0, 6.00)
- added R16: 470R, Resistor_SMD:R_0603_1608Metric, B.Cu at (56.5, 6.00)
- D1, Q1, Q2, Q3, Q4, Q6, Q7, Q9, R1, R10, R11, R12, R13, R2, R3, R4, R5, R6, R7, R8, R9: moved to B.Cu
- moved R7 155.6 mm to (26.0, 23.0)
- moved R11 144.7 mm to (43.0, 14.0), turned to 180 degrees
- moved R5 142.1 mm to (34.0, 22.0)
- moved R8 139.5 mm to (26.0, 28.0)
- moved R10 132.5 mm to (50.0, 14.0), turned to 180 degrees
- moved R6 131.9 mm to (34.0, 27.0)
- moved Q3 121.6 mm to (30.0, 23.0), turned to 180 degrees
- moved R9 119.3 mm to (57.0, 14.0), turned to 180 degrees
- moved Q4 115.4 mm to (30.0, 28.0), turned to 180 degrees
- moved R13 107.1 mm to (75.0, 25.0), turned to 180 degrees
- moved Q6 105.6 mm to (43.0, 10.0), turned to 90 degrees
- moved R12 105.6 mm to (75.0, 29.0), turned to 180 degrees
- moved R3 104.7 mm to (74.0, 17.0), turned to 270 degrees
- moved Q9 98.2 mm to (57.0, 10.0), turned to 90 degrees
- moved Q7 96.8 mm to (50.0, 10.0), turned to 90 degrees
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Connections:
- U1 pad 10: /DISP_c -> /DISP_a
- U1 pad 11: /DISP_d -> /DISP_ca3
- U1 pad 12: /DISP_e -> /DISP_g
- U1 pad 14: /DISP_f -> /DISP_c
- U1 pad 15: /DISP_g -> /DISP_dp
- U1 pad 16: /DISP_dp -> /DISP_d
- U1 pad 17: /DISP_ca1 -> /DISP_e
- U1 pad 19: /DISP_ca2 -> /LED0
- U1 pad 20: /DISP_ca3 -> /LED1
- U1 pad 21: Net-(R3-Pad2) -> PON_SW
- U1 pad 22: PON_SW -> PON_SIG
- U1 pad 24: PON_SIG -> Net-(U1-Pad24)
- U1 pad 27: /LED1 -> Net-(U1-Pad27)
- U1 pad 29: /LED0 -> Net-(U1-Pad29)
- U1 pad 31: /PT0 -> /PT1
- U1 pad 32: /PT1 -> /PT0
- U1 pad 4: Net-(U1-Pad4) -> Net-(R3-Pad2)
- U1 pad 5: Net-(U1-Pad5) -> /DISP_b
- U1 pad 6: Net-(U1-Pad6) -> /DISP_ca1
- U1 pad 7: /DISP_a -> /DISP_ca2
- U1 pad 9: /DISP_b -> /DISP_f
- U2 pad 12: Net-(Q6-Pad3) -> Net-(R14-Pad2)
- U2 pad 8: Net-(Q9-Pad3) -> Net-(R16-Pad2)
- U2 pad 9: Net-(Q7-Pad3) -> Net-(R15-Pad2)
Routing:
- net +3V3: track 0.00 -> 352.5 mm, vias 0 -> 6
- net GND: track 0.00 -> 318.3 mm, vias 0 -> 2
- net +BATT: track 0.00 -> 168.4 mm, vias 0 -> 3
- net /PT1: track 0.00 -> 139.1 mm
- net /PT0: track 0.00 -> 94.1 mm
- net Net-(D3-Pad1): track 0.00 -> 91.2 mm
- net PON_SW: track 0.00 -> 72.5 mm, vias 0 -> 2
- net Net-(D2-Pad1): track 0.00 -> 46.6 mm
- net /DISP_a: track 0.00 -> 44.6 mm
- net /DISP_f: track 0.00 -> 44.3 mm
- net /DISP_b: track 0.00 -> 43.3 mm
- net Net-(SW2-Pad1): track 0.00 -> 42.7 mm
- net PON_SIG: track 0.00 -> 39.3 mm, vias 0 -> 2
- net /DISP_ca3: track 0.00 -> 37.6 mm
- net Net-(BT1-Pad1): track 0.00 -> 37.3 mm
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- added copper zone on F.Cu, net GND
Other:
- outline, holes or cut-outs redrawn
- board text added: "Kick speedometer Ver. 1.0"
- board text added: "Power"
- board text added: "Reset"
